File: scd4x_rf-bm-2652p2.sch (EAGLE design)
At the start: 42 parts, among them IC1 BME280, J5 TYPE-C-31-M-12, Q1 SI2323DS, U1 MCP73831, U2 ap2112k-3.3, U3 XC61CN3202MR-G, U4 SCD41-D-R2, U5 CH340E_MSOP10, U6 SHTC3

Commit message: Add files via upload
Parts:
- added C8: 100nF, discretes-dev:CAP0402
- added R8: 5.1M, RC0402FR-073M6L:RC0402FR-073M6L
Connections:
- net +3V3: now also R8.2
- net DIO15: now also C8.1, R8.1
- net GND: now also C8.2
Other:
- moved on the sheet: BOOT, D1, J1, J2, R4, R5, R7, RST
